Commit message: add robot to world

File: urdf/robo_seeker.urdf.xacro (robot description, xacro)
@@ -1,4 +1,5 @@
 <robot name="robo_seeker"
     xmlns:xacro="http://www.ros.org/wiki/xacro">
+    <xacro:include filename="$(find robo_ball_catcher)/urdf/robo_seeker.gazebo" />
     <link name="robot_footprint"></link>
     <link name='chassis'>
@@ -83,4 +84,42 @@
         </inertial>
     </link>
+    <link name="camera">
+        <visual>
+            <origin xyz="0 0 0" rpy=" 0 0 0"/>
+            <geometry>
+                <box size="0.05 0.05 0.05"/>
+            </geometry>
+        </visual>
+        <collision>
+            <origin xyz="0 0 0" rpy=" 0 0 0"/>
+            <geometry>
+                <box size="0.05 0.05 0.05"/>
+            </geometry>
+        </collision>
+        <inertial>
+            <mass value="0.1"/>
+            <origin xyz="0 0 0" rpy=" 0 0 0"/>
+            <inertia ixx="1e-6" ixy="0" ixz="0" iyy="1e-6" iyz="0" izz="1e-6" />
+        </inertial>
+    </link>
+    <link name="hokuyo">
+        <visual>
+            <origin xyz="0 0 0" rpy=" 0 0 0"/>
+            <geometry>
+                <mesh filename="package://robo_ball_catcher/meshes/hokuyo.dae"/>
+            </geometry>
+        </visual>
+        <collision>
+            <origin xyz="0 0 0.0" rpy=" 0 0 0"/>
+            <geometry>
+                <box size="0.1 0.1 0.1"/>
+            </geometry>
+        </collision>
+        <inertial>
+            <mass value="1e-5"/>
+            <origin xyz="0 0 0.0" rpy=" 0 0 0"/>
+            <inertia ixx="1e-6" ixy="0" ixz="0" iyy="1e-6" iyz="0" izz="1e-6" />
+        </inertial>
+    </link>
     <joint name="robot_footprint_joint" type="fixed">
         <origin xyz="0 0 0" rpy="0 0 0" />
@@ -104,4 +143,16 @@
         <dynamics damping="1.0" friction="1.0"/>
     </joint>
+    <joint type="fixed" name="camera_joint">
+        <origin xyz="0.2 0 0" rpy="0 0 0"/>
+        <child link="camera"/>
+        <parent link="chassis"/>
+        <axis xyz="0 1 0" rpy="0 0 0"/>
+    </joint>
+    <joint type="fixed" name="hokuyo_joint">
+        <origin xyz="0.15 0 0.1" rpy="0 0 0"/>
+        <child link="hokuyo"/>
+        <parent link="chassis"/>
+        <axis xyz="0 1 0" rpy="0 0 0"/>
+    </joint>
     <gazebo reference="chassis">
         <material>Gazebo/Blue</material>
@@ -113,3 +164,6 @@
         <material>Gazebo/Grey</material>
     </gazebo>
+    <gazebo reference="camera">
+        <material>Gazebo/Green</material>
+    </gazebo>
 </robot>
