Commit message: rename package

File: ball_chaser_description/urdf/robo_seeker.urdf.xacro (robot description, xacro)
@@ -1,5 +1,5 @@
 <robot name="robo_seeker"
     xmlns:xacro="http://www.ros.org/wiki/xacro">
-    <xacro:include filename="$(find robo_ball_catcher)/urdf/robo_seeker.gazebo" />
+    <xacro:include filename="$(find ball_chaser_description)/urdf/robo_seeker.gazebo" />
     <link name="robot_footprint"></link>
     <link name='chassis'>
@@ -107,5 +107,5 @@
             <origin xyz="0 0 0" rpy=" 0 0 0"/>
             <geometry>
-                <mesh filename="package://robo_ball_catcher/meshes/hokuyo.dae"/>
+                <mesh filename="package://ball_chaser_description/meshes/hokuyo.dae"/>
             </geometry>
         </visual>

Commit message: add material properties

File: ball_chaser_description/urdf/robo_seeker.urdf.xacro (robot description, xacro)
@@ -20,4 +20,7 @@
                 <box size=".4 .2 .1"/>
             </geometry>
+            <material name="blue">
+                <color rgba="0 0 1 1"/>
+            </material>
         </visual>
         <collision name='back_caster_collision'>
@@ -52,4 +55,7 @@
                 <cylinder radius="0.1" length="0.05"/>
             </geometry>
+            <material name="red">
+                <color rgba="1 0 0 1"/>
+            </material>
         </visual>
         <collision>
@@ -71,4 +77,5 @@
                 <cylinder radius="0.1" length="0.05"/>
             </geometry>
+            <material name="red"/>
         </visual>
         <collision>
@@ -90,4 +97,7 @@
                 <box size="0.05 0.05 0.05"/>
             </geometry>
+            <material name="green">
+                <color rgba="0 1 0 1"/>
+            </material>
         </visual>
         <collision>

Commit message: add ball chaser

File: ball_chaser_description/urdf/robo_seeker.urdf.xacro (robot description, xacro)
@@ -1,5 +1,4 @@
 <robot name="robo_seeker"
     xmlns:xacro="http://www.ros.org/wiki/xacro">
-    <xacro:include filename="$(find ball_chaser_description)/urdf/robo_seeker.gazebo" />
     <link name="robot_footprint"></link>
     <link name='chassis'>
@@ -174,6 +173,85 @@
         <material>Gazebo/Grey</material>
     </gazebo>
+    <gazebo>
+        <plugin name="gazebo_ros_diff_drive" filename="libgazebo_ros_diff_drive.so">
+            <update_rate>10</update_rate>
+            <left_joint>left_wheel_hinge</left_joint>
+            <right_joint>right_wheel_hinge</right_joint>
+            <!-- kinematics -->
+            <wheel_separation>0.4</wheel_separation>
+            <wheel_diameter>0.2</wheel_diameter>
+            <!-- output -->
+            <publish_odom>true</publish_odom>
+            <publish_odom_tf>true</publish_odom_tf>
+            <publish_wheel_tf>true</publish_wheel_tf>
+            <odometry_topic>odom</odometry_topic>
+            <odometry_frame>odom</odometry_frame>
+            <robot_base_frame>robot_footprint</robot_base_frame>
+        </plugin>
+    </gazebo>
     <gazebo reference="camera">
-        <material>Gazebo/Green</material>
+        <material>Gazebo/Grey</material>
+        <sensor name="camera" type="camera">
+            <pose>0 0 0 0 0 0</pose>
+            <visualize>true</visualize>
+            <update_rate>10.0</update_rate>
+            <camera name="realsense_depth_camera">
+                <horizontal_fov>1.46608</horizontal_fov>
+                <image>
+                    <width>800</width>
+                    <height>800</height>
+                    <format>R8G8B8</format>
+                </image>
+                <clip>
+                    <near>0.02</near>
+                    <far>300</far>
+                </clip>
+            </camera>
+            <plugin name="camera_controller" filename="libgazebo_ros_camera.so">
+                <ros>
+                    <namespace>ball_chaser</namespace>
+                    <remapping>image_raw:=camera_img</remapping>
+                </ros>
+                <frame_name>camera</frame_name>
+                <hack_baseline>0.07</hack_baseline>
+                <min_depth>0.05</min_depth>
+                <max_depth>8.0</max_depth>
+            </plugin>
+        </sensor>
+    </gazebo>
+    <!-- hokuyo -->
+    <gazebo reference="hokuyo">
+        <sensor type="ray" name="head_hokuyo_sensor">
+            <pose>0 0 0 0 0 0</pose>
+            <visualize>false</visualize>
+            <update_rate>40</update_rate>
+            <ray>
+                <scan>
+                    <horizontal>
+                        <samples>720</samples>
+                        <resolution>1</resolution>
+                        <min_angle>-1.570796</min_angle>
+                        <max_angle>1.570796</max_angle>
+                    </horizontal>
+                </scan>
+                <range>
+                    <min>0.10</min>
+                    <max>30.0</max>
+                    <resolution>0.01</resolution>
+                </range>
+                <noise>
+                    <type>gaussian</type>
+                    <mean>0.0</mean>
+                    <stddev>0.01</stddev>
+                </noise>
+            </ray>
+            <plugin name="robo_seeker_laserscan" filename="libgazebo_ros_ray_sensor.so">
+                <ros>
+                    <remapping>~/out:=scan</remapping>
+                </ros>
+                <output_type>sensor_msgs/LaserScan</output_type>
+                <frame_name>hokuyo</frame_name>
+            </plugin>
+        </sensor>
     </gazebo>
 </robot>
